File: hardware/easat2.kicad_pcb (KiCad board)
At the start: 2 copper layers, 93 parts, among them P1 CONN_01X02, P2 CONN_01X05, P3 CONN_01X02, P4 CONN_01X02, P5 CONN_01X02, P6 CONN_01X02, P7 CONN_01X02, Q1 FDV301N, U1 LTC3129, U2 LTC3129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

Commit message: Added "AMSAT-EA" to the MPPT PCB silkscreen
Other:
- board text added: "AMSAT-EA"
Changed lines of the file:
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@@
     (area 123.436905 82.891666 167.563096 127.858333)
     (thickness 1.6)
-    (drawings 6)
+    (drawings 7)
     (tracks 614)
     (zones 0)
@@
   (page A4)
   (title_block
-    (title "MPPT Board")
-    (date 2016-09-18)
+    (title EASAT-2)
+    (date 2016-09-19)
     (rev A1)
     (company AMSAT-EA)
@@
     )
   )
+  (gr_text AMSAT-EA (at 138.75 123) (layer B.SilkS)
+    (effects (font (size 2 2) (thickness 0.3)) (justify mirror))
+  )
   (gr_text "EA4GPZ\nEA4GQS\nEA4GVA" (at 151.75 117) (layer B.SilkS)
