File: hardware/MCU/_saved_MCU.sch (KiCad schematic (older format))
At the start: 27 parts, among them P1 CONN_01X05, P2 CONN_01X04, P3 CONN_01X03, U1 MAX6369, U2 DS18B20, U3 PIC18F45K22, Y1 Crystal

Commit message: All footprints added. Need to check them before manufacturing. Placement started
Parts:
- D1: footprint (none) -> LEDs:LED_1206
- U1: footprint TO_SOT_Packages_SMD:SOT-23-6_Handsoldering -> Housings_SOIC:SOIJ-8_5.3x5.3mm_Pitch1.27mm
- Y1: footprint (none) -> Crystals:Crystal_C26-LF_d2.1mm_l6.5mm_Horizontal
- gave numbers to parts that had none: 5
Changed lines of the file:
@@
 F 0 "Y1" H 2900 1900 50  0000 C CNN
 F 1 "Crystal" H 2900 1600 50  0000 C CNN
-F 2 "" H 2900 1750 50  0000 C CNN
+F 2 "Crystals:Crystal_C26-LF_d2.1mm_l6.5mm_Horizontal" H 2900 1750 50  0001 C CNN
 F 3 "" H 2900 1750 50  0000 C CNN
 	1    2900 1750
@@
 F 0 "U1" H 2906 2345 60  0000 C CNN
 F 1 "MAX6369" H 2906 2920 60  0000 C CNN
-F 2 "TO_SOT_Packages_SMD:SOT-23-6_Handsoldering" H 2906 2420 60  0001 C CNN
+F 2 "Housings_SOIC:SOIJ-8_5.3x5.3mm_Pitch1.27mm" H 2906 2420 60  0001 C CNN
 F 3 "" H 2906 2420 60  0001 C CNN
 	1    2906 2420
@@
 F 0 "D1" H 2915 4585 50  0000 C CNN
 F 1 "LED" H 2915 4385 50  0000 C CNN
-F 2 "" H 2915 4485 50  0000 C CNN
+F 2 "LEDs:LED_1206" H 2915 4485 50  0001 C CNN
 F 3 "" H 2915 4485 50  0000 C CNN
 	1    2915 4485
@@
 $EndComp
 $Comp
-L C C?
+L C C8
 U 1 1 58784276
 P 7270 1470
-F 0 "C?" H 7295 1570 50  0000 L CNN
+F 0 "C8" H 7295 1570 50  0000 L CNN
 F 1 "C" H 7295 1370 50  0000 L CNN
 F 2 "Capacitors_SMD:C_1206_HandSoldering" H 7308 1320 50  0001 C CNN
@@
 $EndComp
 $Comp
-L GND #PWR?
+L GND #PWR027
 U 1 1 587842D1
 P 7410 1660
-F 0 "#PWR?" H 7410 1410 50  0001 C CNN
+F 0 "#PWR027" H 7410 1410 50  0001 C CNN
 F 1 "GND" H 7410 1510 50  0000 C CNN
 F 2 "" H 7410 1660 50  0000 C CNN
@@
 $EndComp
 $Comp
-L C C?
+L C C9
 U 1 1 58786231
 P 7560 1470
-F 0 "C?" H 7585 1570 50  0000 L CNN
+F 0 "C9" H 7585 1570 50  0000 L CNN
 F 1 "C" H 7585 1370 50  0000 L CNN
 F 2 "Capacitors_SMD:C_1206_HandSoldering" H 7598 1320 50  0001 C CNN
@@
 $EndComp
 $Comp
-L VCC #PWR?
+L VCC #PWR028
 U 1 1 587868A5
 P 7420 1190
-F 0 "#PWR?" H 7420 1040 50  0001 C CNN
+F 0 "#PWR028" H 7420 1040 50  0001 C CNN
 F 1 "VCC" H 7420 1340 50  0000 C CNN
 F 2 "" H 7420 1190 50  0000 C CNN
@@
 	7560 1280 7560 1320
 Wire Wire Line
-	7560 1620 7270 1620
+	7270 1620 7560 1620
 Wire Wire Line
 	7410 1660 7410 1620
@@
 Connection ~ 7430 1280
 $Comp
-L C C?
+L C C7
 U 1 1 58789C1B
 P 1630 2990
-F 0 "C?" H 1655 3090 50  0000 L CNN
+F 0 "C7" H 1655 3090 50  0000 L CNN
 F 1 "C" H 1655 2890 50  0000 L CNN
 F 2 "Capacitors_SMD:C_1206_HandSoldering" H 1668 2840 50  0001 C CNN
@@
 $EndComp
 $Comp
-L VCC #PWR?
+L VCC #PWR029
 U 1 1 58789D01
 P 1630 2810
-F 0 "#PWR?" H 1630 2660 50  0001 C CNN
+F 0 "#PWR029" H 1630 2660 50  0001 C CNN
 F 1 "VCC" H 1630 2960 50  0000 C CNN
 F 2 "" H 1630 2810 50  0000 C CNN
@@
 $EndComp
 $Comp
-L GND #PWR?
+L GND #PWR030
 U 1 1 58789D60
 P 1630 3190
-F 0 "#PWR?" H 1630 2940 50  0001 C CNN
+F 0 "#PWR030" H 1630 2940 50  0001 C CNN
 F 1 "GND" H 1630 3040 50  0000 C CNN
 F 2 "" H 1630 3190 50  0000 C CNN
@@
 	1630 2810 1630 2840
 $Comp
-L D D?
+L D D2
 U 1 1 5878DC37
 P 8580 3200
-F 0 "D?" H 8580 3300 50  0000 C CNN
+F 0 "D2" H 8580 3300 50  0000 C CNN
 F 1 "D" H 8580 3100 50  0000 C CNN
 F 2 "Diodes_SMD:D_SOD-523" H 8580 3200 50  0001 C CNN
@@
 BUZZER
 $Comp
-L LM358 U?
+L LM358 U4
 U 1 1 587AA4C8
 P 6560 4640
-F 0 "U?" H 6560 4840 50  0000 L CNN
+F 0 "U4" H 6560 4840 50  0000 L CNN
 F 1 "LM358" H 6560 4440 50  0000 L CNN
 F 2 "Housings_SOIC:SOIJ-8_5.3x5.3mm_Pitch1.27mm" H 6560 4640 50  0001 C CNN
@@
 $EndComp
 $Comp
-L LM358 U?
+L LM358 U4
 U 2 1 587AA5C2
 P 8480 4540
-F 0 "U?" H 8480 4740 50  0000 L CNN
+F 0 "U4" H 8480 4740 50  0000 L CNN
 F 1 "LM358" H 8480 4340 50  0000 L CNN
 F 2 "Housings_SOIC:SOIJ-8_5.3x5.3mm_Pitch1.27mm" H 8480 4540 50  0001 C CNN
