File: hardware/MCU/MCU.sch (KiCad schematic (older format))
At the start: 22 parts, among them P1 CONN_01X05, P2 CONN_01X04, P3 CONN_01X03, U1 MAX6369, U2 DS18B20, U3 PIC18F45K22, U4 OP275, Y1 Crystal

Commit message: Some footprints added to MCU components
Parts:
- removed U4: OP275, symbol OP275
- added C? (x3): C, Capacitors_SMD:C_1206_HandSoldering, symbol C
- added D?: D, symbol D
- added U? (x2): LM6161, symbol LM6161
- C1, C2, C3, C5, C6: footprint (none) -> Capacitors_SMD:C_1206_HandSoldering
- R1, R2, R4, R5, R6: footprint (none) -> Resistors_SMD:R_1206_HandSoldering
- R3: value R -> 4K7; footprint (none) -> Resistors_SMD:R_1206_HandSoldering
- U1: footprint (none) -> TO_SOT_Packages_SMD:SOT-23-6_Handsoldering
- U2: footprint (none) -> Housings_SOIC:SOIC-8_3.9x4.9mm_Pitch1.27mm
- U3: footprint (none) -> Housings_SOIC:SOIC-28W_7.5x17.9mm_Pitch1.27mm
Connections:
- wire segments 96 -> 109
Changed lines of the file:
@@
 F 0 "U3" H 6330 2575 60  0000 C CNN
 F 1 "PIC18F45K22" H 6305 3825 60  0000 C CNN
-F 2 "" H 6330 2900 60  0001 C CNN
+F 2 "Housings_SOIC:SOIC-28W_7.5x17.9mm_Pitch1.27mm" H 6330 2900 60  0000 C CNN
 F 3 "" H 6330 2900 60  0001 C CNN
 	1    6330 2900
@@
 F 0 "C2" H 3360 1970 50  0000 L CNN
 F 1 "C_Small" H 3360 1820 50  0000 L CNN
-F 2 "" H 3350 1900 50  0000 C CNN
+F 2 "Capacitors_SMD:C_1206_HandSoldering" H 3350 1900 50  0001 C CNN
 F 3 "" H 3350 1900 50  0000 C CNN
 	1    3350 1900
@@
 F 0 "C1" H 2360 1970 50  0000 L CNN
 F 1 "C_Small" H 2360 1820 50  0000 L CNN
-F 2 "" H 2350 1900 50  0000 C CNN
+F 2 "Capacitors_SMD:C_1206_HandSoldering" H 2350 1900 50  0001 C CNN
 F 3 "" H 2350 1900 50  0000 C CNN
 	1    2350 1900
@@
 F 0 "U1" H 2906 2345 60  0000 C CNN
 F 1 "MAX6369" H 2906 2920 60  0000 C CNN
-F 2 "" H 2906 2420 60  0001 C CNN
+F 2 "TO_SOT_Packages_SMD:SOT-23-6_Handsoldering" H 2906 2420 60  0001 C CNN
 F 3 "" H 2906 2420 60  0001 C CNN
 	1    2906 2420
@@
 F 0 "C3" H 3820 2100 50  0000 L CNN
 F 1 "C" H 3820 1900 50  0000 L CNN
-F 2 "" H 3833 1850 50  0000 C CNN
+F 2 "Capacitors_SMD:C_1206_HandSoldering" H 3833 1850 50  0001 C CNN
 F 3 "" H 3795 2000 50  0000 C CNN
 	1    3795 2000
@@
 F 0 "R2" V 3875 1550 50  0000 C CNN
 F 1 "R" V 3795 1550 50  0000 C CNN
-F 2 "" V 3725 1550 50  0000 C CNN
+F 2 "Resistors_SMD:R_1206_HandSoldering" H 3725 1550 50  0001 C CNN
 F 3 "" H 3795 1550 50  0000 C CNN
 	1    3795 1550
@@
 F 0 "R1" V 2995 4065 50  0000 C CNN
 F 1 "R" V 2915 4065 50  0000 C CNN
-F 2 "" V 2845 4065 50  0000 C CNN
+F 2 "Resistors_SMD:R_1206_HandSoldering" H 2845 4065 50  0001 C CNN
 F 3 "" H 2915 4065 50  0000 C CNN
 	1    2915 4065
@@
 F 0 "U2" H 4105 3995 60  0000 C CNN
 F 1 "DS18B20" H 4105 4495 60  0000 C CNN
-F 2 "" H 4105 4070 60  0001 C CNN
+F 2 "Housings_SOIC:SOIC-8_3.9x4.9mm_Pitch1.27mm" H 4105 4070 60  0000 C CNN
 F 3 "" H 4105 4070 60  0001 C CNN
 	1    4105 4070
@@
 P 4970 2230
 F 0 "R3" V 5050 2230 50  0000 C CNN
-F 1 "R" V 4970 2230 50  0000 C CNN
-F 2 "" V 4900 2230 50  0000 C CNN
+F 1 "4K7" V 4970 2230 50  0000 C CNN
+F 2 "Resistors_SMD:R_1206_HandSoldering" H 4900 2230 50  0001 C CNN
 F 3 "" H 4970 2230 50  0000 C CNN
 	1    4970 2230
@@
 Text Label 7450 2250 0    39   ~ 0
 BUZZER
-Text Label 8940 3035 0    39   ~ 0
-BUZZER
 $Comp
 L GND #PWR015
 U 1 1 5827E8B2
-P 8885 3275
-F 0 "#PWR015" H 8885 3025 50  0001 C CNN
-F 1 "GND" H 8885 3125 50  0000 C CNN
-F 2 "" H 8885 3275 50  0000 C CNN
-F 3 "" H 8885 3275 50  0000 C CNN
-	1    8885 3275
+P 8740 3425
+F 0 "#PWR015" H 8740 3175 50  0001 C CNN
+F 1 "GND" H 8740 3275 50  0000 C CNN
+F 2 "" H 8740 3425 50  0000 C CNN
+F 3 "" H 8740 3425 50  0000 C CNN
+	1    8740 3425
 	1    0    0    -1
 $EndComp
@@
 $EndComp
 $Comp
-L OP275 U4
-U 1 1 586B5CAB
-P 6560 4640
-F 0 "U4" H 6560 4790 50  0000 L CNN
-F 1 "OP275" H 6560 4490 50  0000 L CNN
-F 2 "" H 6460 4690 50  0000 C CNN
-F 3 "" H 6560 4790 50  0000 C CNN
-	1    6560 4640
-	1    0    0    1
-$EndComp
-$Comp
-L OP275 U4
-U 2 1 586B5DE0
-P 8480 4540
-F 0 "U4" H 8480 4690 50  0000 L CNN
-F 1 "OP275" H 8480 4390 50  0000 L CNN
-F 2 "" H 8380 4590 50  0000 C CNN
-F 3 "" H 8480 4690 50  0000 C CNN
-	2    8480 4540
-	1    0    0    1
-$EndComp
-$Comp
 L R R4
 U 1 1 586B5EB4
@@
 F 0 "R4" V 5720 4740 50  0000 C CNN
 F 1 "6,19K" V 5640 4740 50  0000 C CNN
-F 2 "" V 5570 4740 50  0000 C CNN
+F 2 "Resistors_SMD:R_1206_HandSoldering" H 5570 4740 50  0001 C CNN
 F 3 "" H 5640 4740 50  0000 C CNN
 	1    5640 4740
@@
 F 0 "R5" V 7375 4640 50  0000 C CNN
 F 1 "4,99K" V 7295 4640 50  0000 C CNN
-F 2 "" V 7225 4640 50  0000 C CNN
+F 2 "Resistors_SMD:R_1206_HandSoldering" H 7225 4640 50  0001 C CNN
 F 3 "" H 7295 4640 50  0000 C CNN
 	1    7295 4640
@@
 F 0 "R6" V 7795 4640 50  0000 C CNN
 F 1 "6,65K" V 7715 4640 50  0000 C CNN
-F 2 "" V 7645 4640 50  0000 C CNN
+F 2 "Resistors_SMD:R_1206_HandSoldering" H 7645 4640 50  0001 C CNN
 F 3 "" H 7715 4640 50  0000 C CNN
 	1    7715 4640
@@
 F 0 "C4" H 6065 5000 50  0000 L CNN
 F 1 "10nF" H 6065 4800 50  0000 L CNN
-F 2 "" H 6078 4750 50  0000 C CNN
+F 2 "" H 6078 4750 50  0001 C CNN
 F 3 "" H 6040 4900 50  0000 C CNN
 	1    6040 4900
@@
 F 0 "C5" H 8125 4955 50  0000 L CNN
 F 1 "10nF" H 8125 4755 50  0000 L CNN
-F 2 "" H 8138 4705 50  0000 C CNN
+F 2 "Capacitors_SMD:C_1206_HandSoldering" H 8138 4705 50  0001 C CNN
 F 3 "" H 8100 4855 50  0000 C CNN
 	1    8100 4855
@@
 F 0 "C6" H 8575 5590 50  0000 L CNN
 F 1 "10nF" H 8575 5390 50  0000 L CNN
-F 2 "" H 8588 5340 50  0000 C CNN
+F 2 "Capacitors_SMD:C_1206_HandSoldering" H 8588 5340 50  0001 C CNN
 F 3 "" H 8550 5490 50  0000 C CNN
 	1    8550 5490
@@
 	-1   0    0    1
 $EndComp
+$Comp
+L C C?
+U 1 1 58784276
+P 7270 1470
+F 0 "C?" H 7295 1570 50  0000 L CNN
+F 1 "C" H 7295 1370 50  0000 L CNN
+F 2 "Capacitors_SMD:C_1206_HandSoldering" H 7308 1320 50  0001 C CNN
+F 3 "" H 7270 1470 50  0000 C CNN
+	1    7270 1470
+	1    0    0    -1
+$EndComp
+$Comp
+L GND #PWR?
+U 1 1 587842D1
+P 7410 1660
+F 0 "#PWR?" H 7410 1410 50  0001 C CNN
+F 1 "GND" H 7410 1510 50  0000 C CNN
+F 2 "" H 7410 1660 50  0000 C CNN
+F 3 "" H 7410 1660 50  0000 C CNN
+	1    7410 1660
+	1    0    0    -1
+$EndComp
+$Comp
+L C C?
+U 1 1 58786231
+P 7560 1470
+F 0 "C?" H 7585 1570 50  0000 L CNN
+F 1 "C" H 7585 1370 50  0000 L CNN
+F 2 "Capacitors_SMD:C_1206_HandSoldering" H 7598 1320 50  0001 C CNN
+F 3 "" H 7560 1470 50  0000 C CNN
+	1    7560 1470
+	1    0    0    -1
+$EndComp
+$Comp
+L VCC #PWR?
+U 1 1 587868A5
+P 7420 1190
+F 0 "#PWR?" H 7420 1040 50  0001 C CNN
+F 1 "VCC" H 7420 1340 50  0000 C CNN
+F 2 "" H 7420 1190 50  0000 C CNN
+F 3 "" H 7420 1190 50  0000 C CNN
+	1    7420 1190
+	1    0    0    -1
+$EndComp
 Wire Wire Line
 	3050 1750 3350 1750
@@
 	7155 2250 7450 2250
 Wire Wire Line
-	9160 3035 8940 3035
-Wire Wire Line
 	9160 3235 8885 3235
 Wire Wire Line
-	8885 3235 8885 3275
+	8885 3235 8885 3395
 Wire Wire Line
 	3611 2545 3356 2545
@@
 Wire Wire Line
 	3760 5285 3760 5165
+Wire Wire Line
+	7270 1320 7270 1280
+Wire Wire Line
+	7270 1280 7560 1280
+Wire Wire Line
+	7560 1280 7560 1320
+Wire Wire Line
+	7560 1620 7270 1620
+Wire Wire Line
+	7410 1660 7410 1620
+Connection ~ 7410 1620
+Wire Wire Line
+	7420 1190 7420 1280
+Wire Wire Line
+	7420 1280 7430 1280
+Connection ~ 7430 1280
+$Comp
+L C C?
+U 1 1 58789C1B
+P 1630 2990
+F 0 "C?" H 1655 3090 50  0000 L CNN
+F 1 "C" H 1655 2890 50  0000 L CNN
+F 2 "Capacitors_SMD:C_1206_HandSoldering" H 1668 2840 50  0001 C CNN
+F 3 "" H 1630 2990 50  0000 C CNN
+	1    1630 2990
+	1    0    0    -1
+$EndComp
+$Comp
+L VCC #PWR?
+U 1 1 58789D01
+P 1630 2810
+F 0 "#PWR?" H 1630 2660 50  0001 C CNN
+F 1 "VCC" H 1630 2960 50  0000 C CNN
+F 2 "" H 1630 2810 50  0000 C CNN
+F 3 "" H 1630 2810 50  0000 C CNN
+	1    1630 2810
+	1    0    0    -1
+$EndComp
+$Comp
+L GND #PWR?
+U 1 1 58789D60
+P 1630 3190
+F 0 "#PWR?" H 1630 2940 50  0001 C CNN
+F 1 "GND" H 1630 3040 50  0000 C CNN
+F 2 "" H 1630 3190 50  0000 C CNN
+F 3 "" H 1630 3190 50  0000 C CNN
+	1    1630 3190
+	1    0    0    -1
+$EndComp
+Wire Wire Line
+	1630 3190 1630 3140
+Wire Wire Line
+	1630 2810 1630 2840
+$Comp
+L D D?
+U 1 1 5878DC37
+P 8580 3200
+F 0 "D?" H 8580 3300 50  0000 C CNN
+F 1 "D" H 8580 3100 50  0000 C CNN
+F 2 "" H 8580 3200 50  0000 C CNN
+F 3 "" H 8580 3200 50  0000 C CNN
+	1    8580 3200
+	0    1    1    0
+$EndComp
+Wire Wire Line
+	9160 3035 8580 3035
+Wire Wire Line
+	8580 3035 8580 3050
+Wire Wire Line
+	8580 3350 8580 3395
+Wire Wire Line
+	8580 3395 8885 3395
+Wire Wire Line
+	8740 3425 8740 3395
+Connection ~ 8740 3395
+Text Label 8775 3035 0    39   ~ 0
+BUZZER
+$Comp
+L LM6161 U?
+U 1 1 58790D02
+P 6560 4640
+F 0 "U?" H 6560 4940 50  0000 L CNN
+F 1 "LM6161" H 6560 4840 50  0000 L CNN
+F 2 "" H 6610 4840 50  0000 C CNN
+F 3 "" H 6710 4940 50  0000 C CNN
+	1    6560 4640
+	1    0    0    1
+$EndComp
+$Comp
+L LM6161 U?
+U 1 1 58790D79
+P 8480 4540
+F 0 "U?" H 8480 4840 50  0000 L CNN
+F 1 "LM6161" H 8480 4740 50  0000 L CNN
+F 2 "" H 8530 4740 50  0000 C CNN
+F 3 "" H 8630 4840 50  0000 C CNN
+	1    8480 4540
+	1    0    0    1
+$EndComp
 $EndSCHEMATC

Commit message: All footprints added. Need to check them before manufacturing. Placement started
Parts:
- removed U? (x2): LM6161, symbol LM6161
- added U? (x2): LM358, Housings_SOIC:SOIJ-8_5.3x5.3mm_Pitch1.27mm, symbol LM358
- C4: footprint (none) -> Capacitors_SMD:C_1206_HandSoldering
- D?: footprint (none) -> Diodes_SMD:D_SOD-523
- P1: footprint (none) -> Connectors_Terminal_Blocks:TerminalBlock_Pheonix_MPT-2.54mm_5pol
- P2: footprint (none) -> Connectors_Terminal_Blocks:TerminalBlock_Pheonix_MPT-2.54mm_4pol
- P3: footprint (none) -> Connectors_Terminal_Blocks:TerminalBlock_Pheonix_MPT-2.54mm_3pol
- R1: value R -> 470
- SP1: footprint (none) -> Buzzers_Beepers:BUZZER
- Y1: footprint (none) -> Oscillators:Oscillator_DIP-14
Changed lines of the file:
@@
 F 0 "U3" H 6330 2575 60  0000 C CNN
 F 1 "PIC18F45K22" H 6305 3825 60  0000 C CNN
-F 2 "Housings_SOIC:SOIC-28W_7.5x17.9mm_Pitch1.27mm" H 6330 2900 60  0000 C CNN
+F 2 "Housings_SOIC:SOIC-28W_7.5x17.9mm_Pitch1.27mm" H 6330 2900 60  0001 C CNN
 F 3 "" H 6330 2900 60  0001 C CNN
 	1    6330 2900
@@
 F 0 "Y1" H 2900 1900 50  0000 C CNN
 F 1 "Crystal" H 2900 1600 50  0000 C CNN
-F 2 "" H 2900 1750 50  0000 C CNN
+F 2 "Oscillators:Oscillator_DIP-14" H 2900 1750 50  0001 C CNN
 F 3 "" H 2900 1750 50  0000 C CNN
 	1    2900 1750
@@
 P 2915 4065
 F 0 "R1" V 2995 4065 50  0000 C CNN
-F 1 "R" V 2915 4065 50  0000 C CNN
+F 1 "470" V 2915 4065 50  0000 C CNN
 F 2 "Resistors_SMD:R_1206_HandSoldering" H 2845 4065 50  0001 C CNN
 F 3 "" H 2915 4065 50  0000 C CNN
@@
 F 0 "SP1" H 9360 3385 50  0000 C CNN
 F 1 "SPEAKER" H 9360 2885 50  0000 C CNN
-F 2 "" H 9460 3135 50  0000 C CNN
+F 2 "Buzzers_Beepers:BUZZER" H 9460 3135 50  0001 C CNN
 F 3 "" H 9460 3135 50  0000 C CNN
 	1    9460 3135
@@
 F 0 "P2" H 9625 2010 50  0000 C CNN
 F 1 "CONN_01X04" V 9725 1760 50  0000 C CNN
-F 2 "" H 9625 1760 50  0000 C CNN
+F 2 "Connectors_Terminal_Blocks:TerminalBlock_Pheonix_MPT-2.54mm_4pol" H 9625 1760 50  0001 C CNN
 F 3 "" H 9625 1760 50  0000 C CNN
 	1    9625 1760
@@
 F 0 "P3" H 9635 2500 50  0000 C CNN
 F 1 "CONN_01X03" V 9735 2300 50  0000 C CNN
-F 2 "" H 9635 2300 50  0000 C CNN
+F 2 "Connectors_Terminal_Blocks:TerminalBlock_Pheonix_MPT-2.54mm_3pol" H 9635 2300 50  0001 C CNN
 F 3 "" H 9635 2300 50  0000 C CNN
 	1    9635 2300
@@
 F 0 "P1" H 9615 1485 50  0000 C CNN
 F 1 "CONN_01X05" V 9715 1185 50  0000 C CNN
-F 2 "" H 9615 1185 50  0000 C CNN
+F 2 "Connectors_Terminal_Blocks:TerminalBlock_Pheonix_MPT-2.54mm_5pol" H 9615 1185 50  0001 C CNN
 F 3 "" H 9615 1185 50  0000 C CNN
 	1    9615 1185
@@
 F 0 "U2" H 4105 3995 60  0000 C CNN
 F 1 "DS18B20" H 4105 4495 60  0000 C CNN
-F 2 "Housings_SOIC:SOIC-8_3.9x4.9mm_Pitch1.27mm" H 4105 4070 60  0000 C CNN
+F 2 "Housings_SOIC:SOIC-8_3.9x4.9mm_Pitch1.27mm" H 4105 4070 60  0001 C CNN
 F 3 "" H 4105 4070 60  0001 C CNN
 	1    4105 4070
@@
 F 0 "C4" H 6065 5000 50  0000 L CNN
 F 1 "10nF" H 6065 4800 50  0000 L CNN
-F 2 "" H 6078 4750 50  0001 C CNN
+F 2 "Capacitors_SMD:C_1206_HandSoldering" H 6078 4750 50  0001 C CNN
 F 3 "" H 6040 4900 50  0000 C CNN
 	1    6040 4900
@@
 F 0 "D?" H 8580 3300 50  0000 C CNN
 F 1 "D" H 8580 3100 50  0000 C CNN
-F 2 "" H 8580 3200 50  0000 C CNN
+F 2 "Diodes_SMD:D_SOD-523" H 8580 3200 50  0001 C CNN
 F 3 "" H 8580 3200 50  0000 C CNN
 	1    8580 3200
@@
 BUZZER
 $Comp
-L LM6161 U?
-U 1 1 58790D02
+L LM358 U?
+U 1 1 587AA4C8
 P 6560 4640
-F 0 "U?" H 6560 4940 50  0000 L CNN
-F 1 "LM6161" H 6560 4840 50  0000 L CNN
-F 2 "" H 6610 4840 50  0000 C CNN
-F 3 "" H 6710 4940 50  0000 C CNN
+F 0 "U?" H 6560 4840 50  0000 L CNN
+F 1 "LM358" H 6560 4440 50  0000 L CNN
+F 2 "Housings_SOIC:SOIJ-8_5.3x5.3mm_Pitch1.27mm" H 6560 4640 50  0001 C CNN
+F 3 "" H 6560 4640 50  0000 C CNN
 	1    6560 4640
 	1    0    0    1
 $EndComp
 $Comp
-L LM6161 U?
-U 1 1 58790D79
+L LM358 U?
+U 2 1 587AA5C2
 P 8480 4540
-F 0 "U?" H 8480 4840 50  0000 L CNN
-F 1 "LM6161" H 8480 4740 50  0000 L CNN
-F 2 "" H 8530 4740 50  0000 C CNN
-F 3 "" H 8630 4840 50  0000 C CNN
-	1    8480 4540
+F 0 "U?" H 8480 4740 50  0000 L CNN
+F 1 "LM358" H 8480 4340 50  0000 L CNN
+F 2 "Housings_SOIC:SOIJ-8_5.3x5.3mm_Pitch1.27mm" H 8480 4540 50  0001 C CNN
+F 3 "" H 8480 4540 50  0000 C CNN
+	2    8480 4540
 	1    0    0    1
 $EndComp

Commit message: MCU board outline defined. Mechanical holes added. Routing started
Parts:
- added C10: 100nF, Capacitors_SMD:C_1206_HandSoldering, symbol C
- C8: renamed from C?; value C -> 10nF
- C9: renamed from C?; value C -> 100nF
- D1: footprint (none) -> LEDs:LED_1206
- SP1: footprint Buzzers_Beepers:BUZZER -> Buzzers_Beepers:MagneticBuzzer_Kingstate_KCG0601
- U1: footprint TO_SOT_Packages_SMD:SOT-23-6_Handsoldering -> Housings_SOIC:SOIJ-8_5.3x5.3mm_Pitch1.27mm
- Y1: footprint Oscillators:Oscillator_DIP-14 -> Crystals:Crystal_C26-LF_d2.1mm_l6.5mm_Horizontal
- gave numbers to parts that had none: 3
Changed lines of the file:
@@
 F 0 "Y1" H 2900 1900 50  0000 C CNN
 F 1 "Crystal" H 2900 1600 50  0000 C CNN
-F 2 "Oscillators:Oscillator_DIP-14" H 2900 1750 50  0001 C CNN
+F 2 "Crystals:Crystal_C26-LF_d2.1mm_l6.5mm_Horizontal" H 2900 1750 50  0001 C CNN
 F 3 "" H 2900 1750 50  0000 C CNN
 	1    2900 1750
@@
 F 0 "U1" H 2906 2345 60  0000 C CNN
 F 1 "MAX6369" H 2906 2920 60  0000 C CNN
-F 2 "TO_SOT_Packages_SMD:SOT-23-6_Handsoldering" H 2906 2420 60  0001 C CNN
+F 2 "Housings_SOIC:SOIJ-8_5.3x5.3mm_Pitch1.27mm" H 2906 2420 60  0001 C CNN
 F 3 "" H 2906 2420 60  0001 C CNN
 	1    2906 2420
@@
 F 0 "D1" H 2915 4585 50  0000 C CNN
 F 1 "LED" H 2915 4385 50  0000 C CNN
-F 2 "" H 2915 4485 50  0000 C CNN
+F 2 "LEDs:LED_1206" H 2915 4485 50  0001 C CNN
 F 3 "" H 2915 4485 50  0000 C CNN
 	1    2915 4485
@@
 F 0 "SP1" H 9360 3385 50  0000 C CNN
 F 1 "SPEAKER" H 9360 2885 50  0000 C CNN
-F 2 "Buzzers_Beepers:BUZZER" H 9460 3135 50  0001 C CNN
+F 2 "Buzzers_Beepers:MagneticBuzzer_Kingstate_KCG0601" H 9460 3135 50  0001 C CNN
 F 3 "" H 9460 3135 50  0000 C CNN
 	1    9460 3135
@@
 $EndComp
 $Comp
-L C C?
+L C C8
 U 1 1 58784276
 P 7270 1470
-F 0 "C?" H 7295 1570 50  0000 L CNN
-F 1 "C" H 7295 1370 50  0000 L CNN
+F 0 "C8" H 7295 1570 50  0000 L CNN
+F 1 "10nF" H 7295 1370 50  0000 L CNN
 F 2 "Capacitors_SMD:C_1206_HandSoldering" H 7308 1320 50  0001 C CNN
 F 3 "" H 7270 1470 50  0000 C CNN
@@
 $EndComp
 $Comp
-L GND #PWR?
+L GND #PWR027
 U 1 1 587842D1
 P 7410 1660
-F 0 "#PWR?" H 7410 1410 50  0001 C CNN
+F 0 "#PWR027" H 7410 1410 50  0001 C CNN
 F 1 "GND" H 7410 1510 50  0000 C CNN
 F 2 "" H 7410 1660 50  0000 C CNN
@@
 $EndComp
 $Comp
-L C C?
+L C C9
 U 1 1 58786231
 P 7560 1470
-F 0 "C?" H 7585 1570 50  0000 L CNN
-F 1 "C" H 7585 1370 50  0000 L CNN
+F 0 "C9" H 7585 1570 50  0000 L CNN
+F 1 "100nF" H 7585 1370 50  0000 L CNN
 F 2 "Capacitors_SMD:C_1206_HandSoldering" H 7598 1320 50  0001 C CNN
 F 3 "" H 7560 1470 50  0000 C CNN
@@
 $EndComp
 $Comp
-L VCC #PWR?
+L VCC #PWR028
 U 1 1 587868A5
 P 7420 1190
-F 0 "#PWR?" H 7420 1040 50  0001 C CNN
+F 0 "#PWR028" H 7420 1040 50  0001 C CNN
 F 1 "VCC" H 7420 1340 50  0000 C CNN
 F 2 "" H 7420 1190 50  0000 C CNN
@@
 	7560 1280 7560 1320
 Wire Wire Line
-	7560 1620 7270 1620
+	7270 1620 7560 1620
 Wire Wire Line
 	7410 1660 7410 1620
@@
 Connection ~ 7430 1280
 $Comp
-L C C?
+L C C7
 U 1 1 58789C1B
 P 1630 2990
-F 0 "C?" H 1655 3090 50  0000 L CNN
+F 0 "C7" H 1655 3090 50  0000 L CNN
 F 1 "C" H 1655 2890 50  0000 L CNN
 F 2 "Capacitors_SMD:C_1206_HandSoldering" H 1668 2840 50  0001 C CNN
@@
 $EndComp
 $Comp
-L VCC #PWR?
+L VCC #PWR029
 U 1 1 58789D01
 P 1630 2810
-F 0 "#PWR?" H 1630 2660 50  0001 C CNN
+F 0 "#PWR029" H 1630 2660 50  0001 C CNN
 F 1 "VCC" H 1630 2960 50  0000 C CNN
 F 2 "" H 1630 2810 50  0000 C CNN
@@
 $EndComp
 $Comp
-L GND #PWR?
+L GND #PWR030
 U 1 1 58789D60
 P 1630 3190
-F 0 "#PWR?" H 1630 2940 50  0001 C CNN
+F 0 "#PWR030" H 1630 2940 50  0001 C CNN
 F 1 "GND" H 1630 3040 50  0000 C CNN
 F 2 "" H 1630 3190 50  0000 C CNN
@@
 	1630 2810 1630 2840
 $Comp
-L D D?
+L D D2
 U 1 1 5878DC37
 P 8580 3200
-F 0 "D?" H 8580 3300 50  0000 C CNN
+F 0 "D2" H 8580 3300 50  0000 C CNN
 F 1 "D" H 8580 3100 50  0000 C CNN
 F 2 "Diodes_SMD:D_SOD-523" H 8580 3200 50  0001 C CNN
@@
 BUZZER
 $Comp
-L LM358 U?
+L LM358 U4
 U 1 1 587AA4C8
 P 6560 4640
-F 0 "U?" H 6560 4840 50  0000 L CNN
+F 0 "U4" H 6560 4840 50  0000 L CNN
 F 1 "LM358" H 6560 4440 50  0000 L CNN
 F 2 "Housings_SOIC:SOIJ-8_5.3x5.3mm_Pitch1.27mm" H 6560 4640 50  0001 C CNN
@@
 $EndComp
 $Comp
-L LM358 U?
+L LM358 U4
 U 2 1 587AA5C2
 P 8480 4540
-F 0 "U?" H 8480 4740 50  0000 L CNN
+F 0 "U4" H 8480 4740 50  0000 L CNN
 F 1 "LM358" H 8480 4340 50  0000 L CNN
 F 2 "Housings_SOIC:SOIJ-8_5.3x5.3mm_Pitch1.27mm" H 8480 4540 50  0001 C CNN
@@
 	1    0    0    1
 $EndComp
+$Comp
+L C C10
+U 1 1 587B471D
+P 7060 5650
+F 0 "C10" H 7085 5750 50  0000 L CNN
+F 1 "100nF" H 7085 5550 50  0000 L CNN
+F 2 "Capacitors_SMD:C_1206_HandSoldering" H 7098 5500 50  0001 C CNN
+F 3 "" H 7060 5650 50  0000 C CNN
+	1    7060 5650
+	1    0    0    -1
+$EndComp
+$Comp
+L GND #PWR031
+U 1 1 587B47DD
+P 7060 5800
+F 0 "#PWR031" H 7060 5550 50  0001 C CNN
+F 1 "GND" H 7060 5650 50  0000 C CNN
+F 2 "" H 7060 5800 50  0000 C CNN
+F 3 "" H 7060 5800 50  0000 C CNN
+	1    7060 5800
+	1    0    0    -1
+$EndComp
+$Comp
+L VCC #PWR032
+U 1 1 587B4F62
+P 7060 5500
+F 0 "#PWR032" H 7060 5350 50  0001 C CNN
+F 1 "VCC" H 7060 5650 50  0000 C CNN
+F 2 "" H 7060 5500 50  0000 C CNN
+F 3 "" H 7060 5500 50  0000 C CNN
+	1    7060 5500
+	1    0    0    -1
+$EndComp
 $EndSCHEMATC
