File: hardware/MCU/_autosave-MCU.kicad_pcb (KiCad board)
At the start: 2 copper layers, 40 x 40 mm, 46 parts, among them P1 CONN_01X05, P2 CONN_01X04, P3 CONN_01X05, P4 CONN_01X05, U1 MAX6369, U2 TC1262-30VDB, U3 DS18B20, U4 PIC18F45K22, U5 LT6005, Y1 Crystal

Commit message: MCU Version 1.0 lista para fabricación. Ficheros generados.
Other:
- board text added: "nmendi"
Changed lines of the file:
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@@
     (area 8.538096 155.325 57.342857 200.32088)
     (thickness 1.6)
-    (drawings 24)
+    (drawings 25)
     (tracks 820)
     (zones 0)
@@
     (38 B.Mask user hide)
     (39 F.Mask user hide)
-    (40 Dwgs.User user hide)
+    (40 Dwgs.User user)
     (41 Cmts.User user hide)
     (42 Eco1.User user hide)
@@
     (47 F.CrtYd user hide)
     (48 B.Fab user)
-    (49 F.Fab user hide)
+    (49 F.Fab user)
   )
   (setup
@@
     (visible_elements 7FFCFFFF)
     (pcbplotparams
-      (layerselection 0x3ff30_80000001)
+      (layerselection 0x3d0ff_80000001)
       (usegerberextensions false)
       (excludeedgelayer true)
       (linewidth 0.100000)
       (plotframeref false)
-      (viasonmask false)
+      (viasonmask true)
       (mode 1)
       (useauxorigin false)
@@
       (xy -1.552223 2.143973) (xy -2.398889 2.514542) (xy -1.639434 2.527271) (xy -1.010147 2.435593)) (layer F.Fab) (width 0.01))
   )
+  (gr_text nmendi (at 48 172.61) (layer F.Fab)
+    (effects (font (size 1 1) (thickness 0.25)))
+  )
   (gr_line (start 30.13 164.44) (end 29.81 164.61) (layer F.Fab) (width 0.2))

Commit message: - Esquematicos generados - Archivos de fabricacion - BOM para Farnell
Parts:
- removed G?: LOGO, imagenes:amsat-satelite-recortada-fondo-30
- added G***: LOGO, imagenes:amsat-palabra-70, F.Cu at (24.5, 189.5)
- moved FID3 38.7 mm to (44.5, 196.1)
- moved FID2 10.4 mm to (19.5, 190.9)
- moved FID1 3.09 mm to (14.7, 159.6)
