File: hardware/EPS/EPS.sch (KiCad schematic (older format))
At the start: 101 parts, among them J1 Conn_01x11, P1 CONN_01X02, P2 CONN_01X02, P3 CONN_01X02, P4 CONN_01X02, P5 CONN_01X02, P6 CONN_01X02, Q1 BC557, U1 LTC3129, U2 LTC3129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

Commit message: PCB EPS
versión 0
Parts:
- D12, D4, D5, D7, D8: footprint (none) -> Diodes_SMD:D_SOD-523
- L1, L2, L3, L4, L5: footprint Capacitors_SMD:C_1210 -> smini:Murata_LQH32P_footprint; Digikey 490-5348-1-ND -> (none); RS-online (none) -> 106-5317
- P6: footprint Pin_Headers:Pin_Header_Straight_1x02 -> Pin_Headers:Pin_Header_Straight_1x02_Pitch1.27mm
- U1, U2, U3, U4, U5: footprint Housings_SSOP:MSOP-16-1EP-VIA_3x4mm_Pitch0.5mm -> smini:MSOP-16-Pitch0.5mm_LT3129
Changed lines of the file:
@@
 Sheet 1 1
 Title "EASAT-2 EPS"
-Date "2018-05-16"
+Date "2018-05-27"
 Rev "2017-12-27"
 Comp "AMSAT-EA"
 Comment1 "EA4GPZ, updated by EA4GQS, review EA3GHS"
-Comment2 ""
+Comment2 "updated L. Garcés"
 Comment3 ""
 Comment4 ""
@@
 F 0 "U1" H 2350 1950 60  0000 C CNN
 F 1 "LTC3129" H 2950 1650 60  0000 C CNN
-F 2 "Housings_SSOP:MSOP-16-1EP-VIA_3x4mm_Pitch0.5mm" H 3000 1100 60  0001 C CNN
+F 2 "smini:MSOP-16-Pitch0.5mm_LT3129" H 3000 1100 60  0001 C CNN
 F 3 "http://www.linear.com/docs/42736" H 3000 1100 60  0001 C CNN
 	1    3000 1650
@@
 F 0 "L1" V 3100 1000 50  0000 L CNN
 F 1 "10u" V 2950 950 50  0000 L CNN
-F 2 "Capacitors_SMD:C_1210" H 3000 1050 60  0001 C CNN
+F 2 "smini:Murata_LQH32P_footprint" H 3000 1050 60  0001 C CNN
 F 3 "" H 3000 1050 60  0000 C CNN
-F 4 "490-5348-1-ND" V 3000 1050 60  0001 C CNN "Digikey"
+F 4 "106-5317" V 3000 1050 60  0001 C CNN "RS-online"
 	1    3000 1050
 	0    -1   -1   0
@@
 F 0 "P6" H 10850 7150 50  0000 C CNN
 F 1 "CONN_01X02" V 10950 7000 50  0001 C CNN
-F 2 "Pin_Headers:Pin_Header_Straight_1x02" H 10850 7000 60  0001 C CNN
+F 2 "Pin_Headers:Pin_Header_Straight_1x02_Pitch1.27mm" H 10850 7000 60  0001 C CNN
 F 3 "" H 10850 7000 60  0000 C CNN
 	1    10850 7000
@@
 F 0 "U2" H 2350 4150 60  0000 C CNN
 F 1 "LTC3129" H 2950 3850 60  0000 C CNN
-F 2 "Housings_SSOP:MSOP-16-1EP-VIA_3x4mm_Pitch0.5mm" H 3000 3300 60  0001 C CNN
+F 2 "smini:MSOP-16-Pitch0.5mm_LT3129" H 3000 3300 60  0001 C CNN
 F 3 "http://www.linear.com/docs/42736" H 3000 3300 60  0001 C CNN
 	1    3000 3850
@@
 F 0 "L2" V 3100 3200 50  0000 L CNN
 F 1 "10u" V 2950 3150 50  0000 L CNN
-F 2 "Capacitors_SMD:C_1210" H 3000 3250 60  0001 C CNN
+F 2 "smini:Murata_LQH32P_footprint" H 3000 3250 60  0001 C CNN
 F 3 "" H 3000 3250 60  0000 C CNN
-F 4 "490-5348-1-ND" V 3000 3250 60  0001 C CNN "Digikey"
+F 4 "106-5317" V 3000 3250 60  0001 C CNN "RS-online"
 	1    3000 3250
 	0    -1   -1   0
@@
 F 0 "U4" H 8150 1950 60  0000 C CNN
 F 1 "LTC3129" H 8750 1650 60  0000 C CNN
-F 2 "Housings_SSOP:MSOP-16-1EP-VIA_3x4mm_Pitch0.5mm" H 8800 1100 60  0001 C CNN
+F 2 "smini:MSOP-16-Pitch0.5mm_LT3129" H 8800 1100 60  0001 C CNN
 F 3 "http://www.linear.com/docs/42736" H 8800 1100 60  0001 C CNN
 	1    8800 1650
@@
 F 0 "L4" V 8900 1000 50  0000 L CNN
 F 1 "10u" V 8750 950 50  0000 L CNN
-F 2 "Capacitors_SMD:C_1210" H 8800 1050 60  0001 C CNN
+F 2 "smini:Murata_LQH32P_footprint" H 8800 1050 60  0001 C CNN
 F 3 "" H 8800 1050 60  0000 C CNN
-F 4 "490-5348-1-ND" V 8800 1050 60  0001 C CNN "Digikey"
+F 4 "106-5317" V 8800 1050 60  0001 C CNN "RS-online"
 	1    8800 1050
 	0    1    -1   0
@@
 F 0 "U5" H 8150 4150 60  0000 C CNN
 F 1 "LTC3129" H 8750 3850 60  0000 C CNN
-F 2 "Housings_SSOP:MSOP-16-1EP-VIA_3x4mm_Pitch0.5mm" H 8800 3300 60  0001 C CNN
+F 2 "smini:MSOP-16-Pitch0.5mm_LT3129" H 8800 3300 60  0001 C CNN
 F 3 "http://www.linear.com/docs/42736" H 8800 3300 60  0001 C CNN
 	1    8800 3850
@@
 F 0 "L5" V 8900 3200 50  0000 L CNN
 F 1 "10u" V 8750 3150 50  0000 L CNN
-F 2 "Capacitors_SMD:C_1210" H 8800 3250 60  0001 C CNN
+F 2 "smini:Murata_LQH32P_footprint" H 8800 3250 60  0001 C CNN
 F 3 "" H 8800 3250 60  0000 C CNN
-F 4 "490-5348-1-ND" V 8800 3250 60  0001 C CNN "Digikey"
+F 4 "106-5317" V 8800 3250 60  0001 C CNN "RS-online"
 	1    8800 3250
 	0    1    -1   0
@@
 F 0 "U3" H 2350 6200 60  0000 C CNN
 F 1 "LTC3129" H 2950 5900 60  0000 C CNN
-F 2 "Housings_SSOP:MSOP-16-1EP-VIA_3x4mm_Pitch0.5mm" H 3000 5350 60  0001 C CNN
+F 2 "smini:MSOP-16-Pitch0.5mm_LT3129" H 3000 5350 60  0001 C CNN
 F 3 "http://www.linear.com/docs/42736" H 3000 5350 60  0001 C CNN
 	1    3000 5900
@@
 F 0 "L3" V 3100 5250 50  0000 L CNN
 F 1 "10u" V 2950 5200 50  0000 L CNN
-F 2 "Capacitors_SMD:C_1210" H 3000 5300 60  0001 C CNN
+F 2 "smini:Murata_LQH32P_footprint" H 3000 5300 60  0001 C CNN
 F 3 "" H 3000 5300 60  0000 C CNN
-F 4 "490-5348-1-ND" V 3000 5300 60  0001 C CNN "Digikey"
+F 4 "106-5317" V 3000 5300 60  0001 C CNN "RS-online"
 	1    3000 5300
 	0    -1   -1   0
@@
 F 0 "D4" H 5700 1700 50  0000 C CNN
 F 1 "1N4001" H 5700 1500 50  0000 C CNN
-F 2 "" H 5700 1600 50  0001 C CNN
+F 2 "Diodes_SMD:D_SOD-523" H 5700 1600 50  0001 C CNN
 F 3 "" H 5700 1600 50  0001 C CNN
 	1    5700 1600
@@
 F 0 "D7" H 6100 1700 50  0000 C CNN
 F 1 "1N4001" H 6100 1500 50  0000 C CNN
-F 2 "" H 6100 1600 50  0001 C CNN
+F 2 "Diodes_SMD:D_SOD-523" H 6100 1600 50  0001 C CNN
 F 3 "" H 6100 1600 50  0001 C CNN
 	1    6100 1600
@@
 F 0 "D5" H 5700 3900 50  0000 C CNN
 F 1 "1N4001" H 5700 3700 50  0000 C CNN
-F 2 "" H 5700 3800 50  0001 C CNN
+F 2 "Diodes_SMD:D_SOD-523" H 5700 3800 50  0001 C CNN
 F 3 "" H 5700 3800 50  0001 C CNN
 	1    5700 3800
@@
 F 0 "D12" H 5700 5950 50  0000 C CNN
 F 1 "1N4001" H 5700 5750 50  0000 C CNN
-F 2 "" H 5700 5850 50  0001 C CNN
+F 2 "Diodes_SMD:D_SOD-523" H 5700 5850 50  0001 C CNN
 F 3 "" H 5700 5850 50  0001 C CNN
 	1    5700 5850
@@
 F 0 "D8" H 6100 3900 50  0000 C CNN
 F 1 "1N4001" H 6100 3700 50  0000 C CNN
-F 2 "" H 6100 3800 50  0001 C CNN
+F 2 "Diodes_SMD:D_SOD-523" H 6100 3800 50  0001 C CNN
 F 3 "" H 6100 3800 50  0001 C CNN
 	1    6100 3800
@@
 NoConn ~ 8050 2050
 $Comp
-L GND #PWR020
+L GND #PWR019
 U 1 1 5B05FC32
 P 9100 8250
-F 0 "#PWR020" H 9100 8000 50  0001 C CNN
+F 0 "#PWR019" H 9100 8000 50  0001 C CNN
 F 1 "GND" H 9100 8100 50  0000 C CNN
 F 2 "" H 9100 8250 60  0000 C CNN
@@
 GND
 $Comp
-L GND #PWR021
+L GND #PWR020
 U 1 1 5B06F4AD
 P 1400 8150
-F 0 "#PWR021" H 1400 7900 50  0001 C CNN
+F 0 "#PWR020" H 1400 7900 50  0001 C CNN
 F 1 "GND" H 1400 8000 50  0000 C CNN
 F 2 "" H 1400 8150 60  0000 C CNN
@@
 GND
 $Comp
-L PWR_FLAG #FLG022
+L PWR_FLAG #FLG021
 U 1 1 5B089167
 P 1500 7250
-F 0 "#FLG022" H 1500 7325 50  0001 C CNN
+F 0 "#FLG021" H 1500 7325 50  0001 C CNN
 F 1 "PWR_FLAG" H 1500 7400 50  0000 C CNN
 F 2 "" H 1500 7250 50  0001 C CNN
@@
 $EndComp
 $Comp
-L PWR_FLAG #FLG023
+L PWR_FLAG #FLG022
 U 1 1 5B0892A8
 P 2400 7250
-F 0 "#FLG023" H 2400 7325 50  0001 C CNN
+F 0 "#FLG022" H 2400 7325 50  0001 C CNN
 F 1 "PWR_FLAG" H 2400 7400 50  0000 C CNN
 F 2 "" H 2400 7250 50  0001 C CNN
@@
 $EndComp
 $Comp
-L PWR_FLAG #FLG024
+L PWR_FLAG #FLG023
 U 1 1 5B0893E2
 P 3300 7250
-F 0 "#FLG024" H 3300 7325 50  0001 C CNN
+F 0 "#FLG023" H 3300 7325 50  0001 C CNN
 F 1 "PWR_FLAG" H 3300 7400 50  0000 C CNN
 F 2 "" H 3300 7250 50  0001 C CNN
@@
 $EndComp
 $Comp
-L PWR_FLAG #FLG025
+L PWR_FLAG #FLG024
 U 1 1 5B08951C
 P 4200 7250
-F 0 "#FLG025" H 4200 7325 50  0001 C CNN
+F 0 "#FLG024" H 4200 7325 50  0001 C CNN
 F 1 "PWR_FLAG" H 4200 7400 50  0000 C CNN
 F 2 "" H 4200 7250 50  0001 C CNN
@@
 $EndComp
 $Comp
-L PWR_FLAG #FLG026
+L PWR_FLAG #FLG025
 U 1 1 5B089656
 P 5100 7250
-F 0 "#FLG026" H 5100 7325 50  0001 C CNN
+F 0 "#FLG025" H 5100 7325 50  0001 C CNN
 F 1 "PWR_FLAG" H 5100 7400 50  0000 C CNN
 F 2 "" H 5100 7250 50  0001 C CNN
@@
 GND
 $Comp
-L GND #PWR027
+L GND #PWR026
 U 1 1 5B0A2D28
 P 11850 5600
-F 0 "#PWR027" H 11850 5350 50  0001 C CNN
+F 0 "#PWR026" H 11850 5350 50  0001 C CNN
 F 1 "GND" H 11850 5450 50  0000 C CNN
 F 2 "" H 11850 5600 60  0000 C CNN
@@
 Connection ~ 11850 5500
 $Comp
-L PWR_FLAG #FLG028
+L PWR_FLAG #FLG027
 U 1 1 5B0C2BD1
 P 1950 8150
-F 0 "#FLG028" H 1950 8225 50  0001 C CNN
+F 0 "#FLG027" H 1950 8225 50  0001 C CNN
 F 1 "PWR_FLAG" H 1950 8300 50  0000 C CNN
 F 2 "" H 1950 8150 50  0001 C CNN
