File: hardware/EPS/EPS.kicad_pcb (KiCad board)
At the start: 2 copper layers, 95 parts, among them J1 Conn_01x11, P1 CONN_01X02, P2 CONN_01X02, P3 CONN_01X02, P4 CONN_01X02, P5 CONN_01X02, Q1 BC557, U1 LTC3129, U2 LTC3129, U3 LTC3129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

Commit message: PCB EPS
versión 0
Parts:
- added D12: 1N4001, Diodes_SMD:D_SOD-523, F.Cu at (128.5, 133.0)
- added D4: 1N4001, Diodes_SMD:D_SOD-523, F.Cu at (90.0, 133.0)
- added D5: 1N4001, Diodes_SMD:D_SOD-523, F.Cu at (110.0, 133.0)
- added D7: 1N4001, Diodes_SMD:D_SOD-523, F.Cu at (115.8, 125.0)
- added D8: 1N4001, Diodes_SMD:D_SOD-523, F.Cu at (97.3, 125.0)
- added P6: CONN_01X02, Pin_Headers:Pin_Header_Straight_1x02_Pitch1.27mm, F.Cu at (76.4, 110.8)
- L1, L2, L3, L4, L5: footprint Capacitors_SMD:C_1210 -> smini:Murata_LQH32P_footprint
- U1, U2, U3, U4, U5: footprint Housings_SSOP:MSOP-16-1EP-VIA_3x4mm_Pitch0.5mm -> smini:MSOP-16-Pitch0.5mm_LT3129
- moved C10 81.6 mm to (78.0, 146.0), turned to 180 degrees
- moved R4 80.0 mm to (81.0, 148.0), turned to 270 degrees
- moved C1 79.4 mm to (78.0, 141.5), turned to 270 degrees
- moved R5 77.9 mm to (83.5, 148.0), turned to 90 degrees
- moved P1 77.7 mm to (77.5, 136.5), turned to 270 degrees
- moved R1 76.3 mm to (77.5, 133.0), turned to 270 degrees
- moved J1 75.9 mm to (76.3, 128.5), turned to 180 degrees
- moved R11 75.9 mm to (86.0, 148.0), turned to 270 degrees
- moved U1 74.4 mm to (84.0, 142.0), turned to 90 degrees
- moved C4 74.2 mm to (81.2, 136.3), turned to 180 degrees
- moved R10 73.0 mm to (88.5, 146.5), turned to 270 degrees
- moved R22 71.7 mm to (80.7, 128.4), turned to 270 degrees
- moved C16 70.9 mm to (91.0, 146.5), turned to 270 degrees
- moved L1 70.5 mm to (83.8, 133.0)
- moved D11 69.8 mm to (80.6, 121.5), turned to 270 degrees
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Connections:
- J1 pad 2: GND -> PTT
- Q1 pad 2: Net-(Q1-Pad2) -> PTT
- R35 pad 1: Net-(Q1-Pad2) -> VBUS
- R35 pad 2: GND -> PTT
- U1 pad 6: (no net) -> GND
- U1 pad 7: (no net) -> GND
- U1 pad 9: Net-(U1-Pad9) -> (no net)
- U2 pad 6: (no net) -> GND
- U2 pad 7: (no net) -> GND
- U2 pad 9: Net-(U2-Pad9) -> (no net)
- U3 pad 6: (no net) -> GND
- U3 pad 7: (no net) -> GND
- U3 pad 9: Net-(U3-Pad9) -> (no net)
- U4 pad 6: (no net) -> GND
- U4 pad 7: (no net) -> GND
- U4 pad 9: Net-(U4-Pad9) -> (no net)
- U5 pad 6: (no net) -> GND
- U5 pad 7: (no net) -> GND
- U5 pad 9: Net-(U5-Pad9) -> (no net)
Routing:
- net GND: track 0.00 -> 191.7 mm, vias 0 -> 5
- net Net-(D12-Pad1): track 0.00 -> 60.9 mm
- net PV-X_OUT: track 0.00 -> 58.4 mm, vias 0 -> 2
- net PV+Z_OUT: track 0.00 -> 45.0 mm, vias 0 -> 1
- net PV-Y_OUT: track 0.00 -> 38.8 mm, vias 0 -> 1
- net VBUS: track 0.00 -> 32.5 mm
- net I_BATT_D: track 0.00 -> 30.5 mm, vias 0 -> 2
- net PV+Y_OUT: track 0.00 -> 26.1 mm, vias 0 -> 1
- net PV-X_IN: track 0.00 -> 22.2 mm, vias 0 -> 2
- net PV-Y_IN: track 0.00 -> 22.2 mm, vias 0 -> 2
- net PV+Y_IN: track 0.00 -> 22.2 mm, vias 0 -> 2
- net PV+Z_IN: track 0.00 -> 22.1 mm, vias 0 -> 2
- net PV+X_IN: track 0.00 -> 22.1 mm, vias 0 -> 2
- net PTT: track 0.00 -> 21.1 mm, vias 0 -> 2
- net Net-(C20-Pad1): track 0.00 -> 19.0 mm
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- added copper zone on B.Cu, net GND
- added copper zone on F.Cu, net GND
- added copper zone on F.Cu, net Net-(C13-Pad2)
- added copper zone on F.Cu, net Net-(C14-Pad2)
- added copper zone on F.Cu, net Net-(C15-Pad2)
- added copper zone on F.Cu, net Net-(C19-Pad1)
- added copper zone on F.Cu, net Net-(C20-Pad1)
- added copper zone on F.Cu, net Net-(C26-Pad1)
- added copper zone on F.Cu, net Net-(C26-Pad2)
- added copper zone on F.Cu, net Net-(C27-Pad1)
- added copper zone on F.Cu, net Net-(C27-Pad2)
- added copper zone on F.Cu, net Net-(C28-Pad1)
- added copper zone on F.Cu, net Net-(C28-Pad2)
- added copper zone on F.Cu, net Net-(C29-Pad1)
- added copper zone on F.Cu, net Net-(C29-Pad2)
- added copper zone on F.Cu, net Net-(C4-Pad1)
- added copper zone on F.Cu, net Net-(C4-Pad2)
- added copper zone on F.Cu, net Net-(C5-Pad1)
- added copper zone on F.Cu, net Net-(C5-Pad2)
- added copper zone on F.Cu, net Net-(C6-Pad1)
- added copper zone on F.Cu, net Net-(C6-Pad2)
- added copper zone on F.Cu, net Net-(C7-Pad1)
- added copper zone on F.Cu, net Net-(C7-Pad2)
- added copper zone on F.Cu, net Net-(C8-Pad1)
- added copper zone on F.Cu, net Net-(C8-Pad2)
- added copper zone on F.Cu, net Net-(C9-Pad1)
- added copper zone on F.Cu, net Net-(C9-Pad2)
- added copper zone on F.Cu, net Net-(D1-Pad1)
- added copper zone on F.Cu, net Net-(D10-Pad1)
- added copper zone on F.Cu, net Net-(D12-Pad1)
- added copper zone on F.Cu, net Net-(D12-Pad2)
- added copper zone on F.Cu, net Net-(D2-Pad1)
- added copper zone on F.Cu, net Net-(D7-Pad2)
- added copper zone on F.Cu, net PV+X_IN
- added copper zone on F.Cu, net PV+Y_IN
- added copper zone on F.Cu, net PV+Z_IN
- added copper zone on F.Cu, net PV-X_IN
- added copper zone on F.Cu, net PV-Y_IN
Other:
- net class Default: trace_width 0.25 -> 0.5
- net class LT3129 added: clearance 0.175, trace_width 0.305, via_dia 0.3, via_drill 0.2
- net class LT3129_outputs added: clearance 0.25, trace_width 1.25, via_dia 0.6, via_drill 0.4
- net class Vbus added: clearance 0.25, trace_width 1, via_dia 0.6, via_drill 0.4
- rule trace_min: 0.2 -> 0.3
- rule via_min_drill: 0.3 -> 0.2
- rule via_min_size: 0.4 -> 0.3

Commit message: Actualización PCB EPS
Parts:
- added ?: 1pin, Connectors:1pin, F.Cu at (166.0, 69.0)
- added ?: 1pin, Connectors:1pin, F.Cu at (166.0, 116.0)
- added ?: 1pin, Connectors:1pin, F.Cu at (114.0, 116.0)
- added ?: 1pin, Connectors:1pin, F.Cu at (114.0, 69.0)
- moved C21 51.9 mm to (119.9, 92.2)
- moved C28 51.9 mm to (161.8, 85.6)
- moved C31 51.9 mm to (130.3, 81.4)
- moved C30 51.9 mm to (118.8, 76.8)
- moved Q1 51.9 mm to (124.8, 85.7)
- moved R23 51.9 mm to (121.8, 80.4)
- moved R24 51.9 mm to (125.7, 80.3)
- moved R25 51.9 mm to (116.6, 76.8)
- moved R35 51.9 mm to (130.3, 85.5)
- moved RLIM1 51.9 mm to (121.8, 85.1)
- moved C1 51.9 mm to (115.2, 105.4)
- moved C10 51.9 mm to (115.2, 109.9)
- moved C11 51.9 mm to (135.2, 109.9)
- moved C13 51.9 mm to (126.7, 105.4)
- moved C14 51.9 mm to (146.7, 105.4)
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Other:
- board outline added: 60 x 55 mm
- board text added: "AMSAT-EA (2018)"
- board text added: "EPS v1.0 AMSAT-EA (2018)"
